Commit message: 把a1换成了自己的四足模型，成功MPC+QP+SLOP

File: src/quadruped/urdf/quadruped_mdf_inertia.urdf (robot description, URDF)
Before this commit: robot quadruped, 17 links, 16 joints
Links:
- link LbL1: mass 0.2020892 -> 0.0520892
- link LbL2: mass 0.203684 -> 0.053684
- link LbL3: mass 0.2012147 -> 0.053684
- link LbL4: mass 0.2012147 -> 0.053684
- link LfL1: mass 0.2020892 -> 0.0520892
- link LfL2: mass 0.203684 -> 0.053684
- link LfL3: mass 0.2012147 -> 0.053684
- link LfL4: mass 0.2012147 -> 0.053684
- link RbL1: mass 0.2020892 -> 0.0520892
- link RbL2: mass 0.203684 -> 0.053684
- link RbL3: mass 0.2012147 -> 0.053684
- link RbL4: mass 0.2012147 -> 0.053684
- link RfL1: mass 0.2020892 -> 0.0520892
- link RfL2: mass 0.203684 -> 0.053684
- link RfL3: mass 0.2012147 -> 0.053684
- link RfL4: mass 0.2012147 -> 0.053684

File: src/quadruped/urdf/quadruped_ori_inertia.urdf (robot description, URDF)
Before this commit: robot quadruped, 18 links, 17 joints
Links:
- removed link world
- link base_link: mass 6.2588 -> 16
Joints:
- removed joint fix
