Commit message: 加入了老程序的上下台阶功能

File: src/hexapod_description2/urdf/hexapod_description2_mdf_init.urdf (robot description, URDF)
Before this commit: robot hexapod_description2, 19 links, 18 joints
Links:
- added link world
Joints:
- added joint fix: type fixed, parent world, child base_link, origin xyz=0 0 0.5 rpy=0 0 0

Commit message: 开始接入硬件

File: src/hexapod_description2/urdf/hexapod_description2_mdf_init.urdf (robot description, URDF)
Before this commit: robot hexapod_description2, 20 links, 19 joints
Links:
- removed link world
Joints:
- removed joint fix
